Commit message: arm control working but marker publisher not

File: urdf/robot.xacro (robot description, xacro)
@@ -264,18 +264,18 @@
 	<link name="camera">
 		<collision>
-			<origin xyz="0 0 0.025" rpy="0 0 0"/>
-			<geometry>
-				<box size="0.02 0.02 0.02"/>
-			</geometry>
-		</collision>
-		<visual>
-			<origin xyz="0 0 0.025" rpy="0 0 0"/>
-			<geometry>
-				<box size="0.02 0.02 0.02"/>
+			<origin xyz="0 0 0" rpy="0 0 0"/>
+			<geometry>
+				<box size="0.05 0.05 0.05"/>
+			</geometry>
+		</collision>
+		<visual>
+			<origin xyz="0 0 0" rpy="0 0 0"/>
+			<geometry>
+				<box size="0.05 0.05 0.05"/>
 			</geometry>
 			<material name="white"/>
 		</visual>
 		<inertial>
-			<mass value="0" />
+			<mass value="${camera_mass}" />
 			<origin xyz="0 0 0" rpy="0 0 0"/>
 			<inertia ixx="0" ixy="0" ixz="0" iyy="0" iyz="0" izz="0" />
@@ -355,6 +355,6 @@
 	</joint> -->
 	<joint name="camera_joint" type="fixed">
-		<axis xyz="0 0 0" />
-		<origin xyz="0 0.0 0.07" rpy="0 0 0"/>
+		<axis xyz="0 1 0" />
+		<origin xyz="0 0.0 0.08" rpy="0 0 0"/>
 		<parent link="arm_L3"/>
 		<child link="camera"/>

Commit message: the map not built coorectly yet but everything else is working

File: urdf/robot.xacro (robot description, xacro)
@@ -355,5 +355,5 @@
 	</joint> -->
 	<joint name="camera_joint" type="fixed">
-		<axis xyz="0 1 0" />
+		<axis xyz="0 0 0" />
 		<origin xyz="0 0.0 0.08" rpy="0 0 0"/>
 		<parent link="arm_L3"/>
